File: kicad/v1.1/usynth.sch (KiCad schematic (older format))
At the start: 54 parts, among them J1 MAIN_CONN, J2 AVR-ISP-6, J3 LINE_OUT, J4 MIDI_IN, U1 ATmega328-AU, U2 MCP4921, U3 TL431DBZ, U4 MCP6001, U5 6N137, U6 L78L05_SO8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

Commit message: Export gerber files, add PCB version suitable for JLC PCB SMT assembly
Parts:
- U2: footprint Package_SO:MSOP-8_3x3mm_P0.65mm -> Package_SO:SOIC-8_3.9x4.9mm_P1.27mm
Changed lines of the file:
@@
 F 0 "U2" H 5000 4650 50  0000 L CNN
 F 1 "MCP4921" H 5000 4750 50  0000 L CNN
-F 2 "Package_SO:MSOP-8_3x3mm_P0.65mm" H 5550 4850 50  0001 C CNN
+F 2 "Package_SO:SOIC-8_3.9x4.9mm_P1.27mm" H 5550 4850 50  0001 C CNN
 F 3 "http://ww1.microchip.com/downloads/en/DeviceDoc/22248a.pdf" H 5550 4850 50  0001 C CNN
 	1    4550 4950
